Commit message: commit_

File: blimp_description/urdf/description_property.xacro (robot description, xacro)
@@ -19,6 +19,6 @@
 	<!-- mass [kg] -->
 	<!-- Modified mass for convenience -->
-	<xacro:property name="mass_blimp_body" value="4.622" />
-	<xacro:property name="mass_blimp_body_without_gas" value="2.90" />
+	<xacro:property name="mass_blimp_body" value="4.622" /> <!--default: 4.622 -->
+	<xacro:property name="mass_blimp_body_without_gas" value="2.9" /> <!--default: 2.90 -->
 	<xacro:property name="mass_gondola_body" value="1.105" /> <!--battery: 0.51kg + body:0.595kg = 1.105-->
 	<!--<xacro:property name="mass_gondola_body" value="0.845" />--> <!--battery: 0.25kg + body:0.595kg = 0.845-->
@@ -31,9 +31,9 @@
 	<xacro:property name="mass_bot_rud_part1" value="0.410" /> <!--part1: 0.120kg + wire: 0.290kg = 0.410 -->
 	<xacro:property name="mass_bot_rud_motor" value="0.127" />
-	<xacro:property name="mass_ballast" value="0.6" /> <!--default: 0.4 -->
+	<xacro:property name="mass_ballast" value="0.6" /> <!--default: 0.6 -->
 	<!-- geometry [m] -->
-	<xacro:property name="radius_blimp_body" value="1.00"/>
-	<xacro:property name="length_blimp_body" value="5.00"/>
-	<xacro:property name="volume_blimp_body" value="10.472"/>
+	<xacro:property name="radius_blimp_body" value="1"/> <!--default: 1 -->
+	<xacro:property name="length_blimp_body" value="5"/> <!--default: 5 -->
+	<xacro:property name="volume_blimp_body" value="10.472 "/> <!--default: 10.472 -->
 	<xacro:property name="length_blimp_skin" value="0.0002"/>
 	<xacro:property name="length_gondola_body" value="0.420"/>
